File: Assignment_1/Assignment 1.kicad_pcb (KiCad board)
At the start: 2 copper layers, 92.5 x 66.5 mm, 17 parts, among them J4 Jack-DC, J5 Screw_Terminal_01x02, J6 Screw_Terminal_01x02, SW2 1825163-2, T2 TY-311P, U1 LM7805_TO220, U2 LM317_TO-220, X1 AC Jack

Commit message: Update layout of all assignments - P2
Parts:
- added G***: LOGO, Logo:logo, B.Cu at (176.0, 42.5)
Routing:
- net /5V: track 26.0 -> 18.6 mm
Other:
- board text added: "Name: Ahmed Atef Nasr ID: 1471804251201"
