File: Assignment_2/P2/L7 - P1.kicad_pcb (KiCad board)
At the start: 2 copper layers, 37.5 x 20.5 mm, 9 parts, among them J1 Conn_01x03_Pin, U1 LM358

Commit message: Update layout of all assignments - P2
Parts:
- added G***: LOGO, Logo:logo, B.Cu at (140.5, 70.5)
Other:
- board text added: "Name: Ahmed Atef Nasr ID: 1471804251201"
